File: OPEnS-RTC-1.1.sch (EAGLE design)
At the start: 58 parts, among them U1 FRAM, U2 DS3231ST&R

Commit message: Revised components and labels.
Added documentation (with BoM) as a .docx and .pdf. Swapped pins on JST connectors. Removed pointless pullup resistor, added current limiting resistor for LED. Swapped 2mm barrel jack for 0.9mm x 3.2mm barrel jack. Combined components into OPEnS-RTC.lbr.
Parts:
- removed R3: 10k, rcl:R-US_R0805
- FEATHER: device bluefruit_m0:BLUEFRUIT_M0 -> OPEnS-RTC:BLUEFRUIT_M0
- HV_IN: value (none) -> PJ-028-SMT-TR; device adafruit:DCBARRELSMT -> OPEnS-RTC:PJ-028-SMT-TR
Connections:
- removed net N$20: FEATHER.10, SJ3.2
- new net N$17: FEATHER.9, SJ3.2
- net +4.1V: no longer R3.2
- net GND: now also HV_IN.2, HV_IN.3; no longer HV_IN.GND, HV_IN.GNDBREAK
- net VCC_HV: now also HV_IN.1; no longer HV_IN.PWR
- net V_LATCH: no longer R3.1
Other:
- note added: "Bulk"
- note added: "Change value as needed"
- note added: "Decoupling"
- note added: "I2C Pullups"
- note added: "Low-pass"
- note added: "set value based on expected noise"
Changed lines of the file:
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@@
 <part name="R2" library="rcl" library_urn="urn:adsk.eagle:library:334" deviceset="R-US_" device="R0805" package3d_urn="urn:adsk.eagle:package:23553/2" value="500"/>
 <part name="FET_P1" library="transistor-small-signal" library_urn="urn:adsk.eagle:library:401" deviceset="BSS84" device="" package3d_urn="urn:adsk.eagle:package:28738/2"/>
-<part name="R3" library="rcl" library_urn="urn:adsk.eagle:library:334" deviceset="R-US_" device="R0805" package3d_urn="urn:adsk.eagle:package:23553/2" value="10k"/>
 <part name="R4" library="rcl" library_urn="urn:adsk.eagle:library:334" deviceset="R-US_" device="R0805" package3d_urn="urn:adsk.eagle:package:23553/2" value="500"/>
 <part name="FET_N2" library="adafruit" deviceset="MOSFET-N" device="REFLOW"/>
@@
 <part name="R8" library="rcl" library_urn="urn:adsk.eagle:library:334" deviceset="R-US_" device="R0805" package3d_urn="urn:adsk.eagle:package:23553/2" value="10k"/>
 <part name="FET_P3" library="transistor-small-signal" library_urn="urn:adsk.eagle:library:401" deviceset="BSS84" device="" package3d_urn="urn:adsk.eagle:package:28738/2"/>
-<part name="SUPPLY1" library="supply2" library_urn="urn:adsk.eagle:library:372" deviceset="+4.1V" device=""/>
 <part name="SUPPLY2" library="supply2" library_urn="urn:adsk.eagle:library:372" deviceset="+4.1V" device=""/>
 <part name="SUPPLY3" library="supply2" library_urn="urn:adsk.eagle:library:372" deviceset="+4.1V" device=""/>
@@
 <part name="TEST5" library="pinhead" library_urn="urn:adsk.eagle:library:325" deviceset="PINHD-1X1" device="" package3d_urn="urn:adsk.eagle:package:22485/2"/>
 <part name="TEST6" library="pinhead" library_urn="urn:adsk.eagle:library:325" deviceset="PINHD-1X1" device="" package3d_urn="urn:adsk.eagle:package:22485/2"/>
-<part name="FEATHER" library="bluefruit_m0" deviceset="BLUEFRUIT_M0" device=""/>
+<part name="FEATHER" library="OPEnS-RTC" deviceset="BLUEFRUIT_M0" device=""/>
 <part name="GND15" library="supply1" library_urn="urn:adsk.eagle:library:371" deviceset="GND" device=""/>
 <part name="+3V5" library="supply1" library_urn="urn:adsk.eagle:library:371" deviceset="+3V3" device=""/>
@@
 <part name="GND19" library="supply1" library_urn="urn:adsk.eagle:library:371" deviceset="GND" device=""/>
 <part name="SUPPLY4" library="supply2" library_urn="urn:adsk.eagle:library:372" deviceset="+4.1V" device=""/>
-<part name="HV_IN" library="adafruit" deviceset="DCBARREL" device="SMT"/>
 <part name="LV_IN" library="adafruit" deviceset="JST_2PIN" device="-SMT"/>
 <part name="GND20" library="supply1" library_urn="urn:adsk.eagle:library:371" deviceset="GND" device=""/>
@@
 <part name="GND22" library="supply1" library_urn="urn:adsk.eagle:library:371" deviceset="GND" device=""/>
 <part name="R5" library="rcl" library_urn="urn:adsk.eagle:library:334" deviceset="R-US_" device="R0805" package3d_urn="urn:adsk.eagle:package:23553/2" value="50"/>
+<part name="HV_IN" library="OPEnS-RTC" deviceset="PJ-028-SMT-TR" device=""/>
 </parts>
 <sheets>
@@
 <text x="104.14" y="-22.86" size="2.54" layer="97">OPEnS Lab OSU</text>
 <text x="106.68" y="-43.18" size="2.54" layer="97">1</text>
-<text x="170.18" y="-43.18" size="2.54" layer="97">1</text>
+<text x="170.18" y="-43.18" size="2.54" layer="97">2</text>
+<text x="70.612" y="6.35" size="2.54" layer="97" font="vector">Low-pass</text>
+<text x="70.358" y="2.54" size="2.54" layer="97" font="vector">set value based on expected noise</text>
 </plain>
 <instances>
@@
 <attribute name="VALUE" x="15.24" y="71.12" size="1.778" layer="96"/>
 </instance>
-<instance part="R3" gate="G$1" x="-22.86" y="60.96" smashed="yes" rot="R90">
-<attribute name="NAME" x="-24.3586" y="57.15" size="1.778" layer="95" rot="R90"/>
-<attribute name="VALUE" x="-19.558" y="57.15" size="1.778" layer="96" rot="R90"/>
-</instance>
 <instance part="R4" gate="G$1" x="-10.16" y="53.34" smashed="yes" rot="R180">
 <attribute name="NAME" x="-6.35" y="51.8414" size="1.778" layer="95" rot="R180"/>
@@
 <attribute name="NAME" x="76.2" y="119.38" size="1.778" layer="95"/>
 <attribute name="VALUE" x="76.2" y="116.84" size="1.778" layer="96"/>
-</instance>
-<instance part="SUPPLY1" gate="P" x="-22.86" y="71.12" smashed="yes">
-<attribute name="VALUE" x="-24.765" y="74.295" size="1.778" layer="96"/>
 </instance>
 <instance part="SUPPLY2" gate="P" x="12.7" y="86.36" smashed="yes">
@@
 <pinref part="R4" gate="G$1" pin="2"/>
 <wire x1="-15.24" y1="53.34" x2="-22.86" y2="53.34" width="0.1524" layer="91"/>
-<pinref part="R3" gate="G$1" pin="1"/>
-<wire x1="-22.86" y1="53.34" x2="-22.86" y2="55.88" width="0.1524" layer="91"/>
 <wire x1="-22.86" y1="53.34" x2="-35.56" y2="53.34" width="0.1524" layer="91"/>
 <junction x="-22.86" y="53.34"/>
@@
 <net name="+4.1V" class="0">
 <segment>
-<pinref part="R3" gate="G$1" pin="2"/>
-<wire x1="-22.86" y1="66.04" x2="-22.86" y2="68.58" width="0.1524" layer="91"/>
-<pinref part="SUPPLY1" gate="P" pin="+4.1V"/>
-</segment>
-<segment>
 <pinref part="FET_P1" gate="G$1" pin="S"/>
 <wire x1="12.7" y1="78.74" x2="12.7" y2="83.82" width="0.1524" layer="91"/>
@@
 <plain>
 <text x="187.96" y="-66.04" size="2.54" layer="97">2</text>
-<text x="248.92" y="-66.04" size="2.54" layer="97">1</text>
+<text x="248.92" y="-66.04" size="2.54" layer="97">2</text>
 <text x="157.48" y="-48.26" size="2.54" layer="97">mitchell nelke OPEnS Lab OSU</text>
+<text x="86.868" y="109.728" size="2.54" layer="97" font="vector">Decoupling</text>
+<text x="-10.16" y="27.94" size="2.54" layer="97" font="vector" rot="R90">Decoupling</text>
+<text x="141.732" y="32.004" size="2.54" layer="97" font="vector">Decoupling</text>
+<text x="120.904" y="31.242" size="2.54" layer="97" font="vector">Bulk</text>
+<text x="107.442" y="-59.436" size="2.54" layer="97" font="vector">I2C Pullups</text>
+<text x="107.188" y="-62.992" size="2.54" layer="97" font="vector">Change value as needed</text>
 </plain>
 <instances>
@@
 <attribute name="VALUE" x="40.64" y="-36.83" size="1.778" layer="96" rot="R180"/>
 </instance>
-<instance part="SJ3" gate="1" x="96.52" y="-43.18" smashed="yes" rot="R180">
-<attribute name="NAME" x="96.52" y="-38.1" size="1.778" layer="95" rot="R180"/>
-<attribute name="VALUE" x="99.06" y="-39.37" size="1.778" layer="96" rot="R180"/>
+<instance part="SJ3" gate="1" x="111.76" y="-43.18" smashed="yes" rot="R180">
+<attribute name="NAME" x="111.76" y="-38.1" size="1.778" layer="95" rot="R180"/>
+<attribute name="VALUE" x="114.3" y="-39.37" size="1.778" layer="96" rot="R180"/>
 </instance>
 <instance part="HV_SW" gate="G$1" x="248.92" y="25.4" smashed="yes">
@@
 <attribute name="VALUE" x="187.325" y="5.715" size="1.778" layer="96" rot="R90"/>
 </instance>
-<instance part="HV_IN" gate="G$1" x="170.18" y="-17.78" smashed="yes">
-<attribute name="NAME" x="165.1" y="-12.7" size="1.27" layer="95"/>
-<attribute name="VALUE" x="165.1" y="-22.86" size="1.27" layer="96"/>
-</instance>
 <instance part="LV_IN" gate="G$1" x="243.84" y="-20.32" smashed="yes">
 <attribute name="NAME" x="237.49" y="-14.605" size="1.778" layer="95"/>
@@
 <instance part="GND22" gate="1" x="193.04" y="45.72" smashed="yes" rot="R270">
 <attribute name="VALUE" x="190.5" y="48.26" size="1.778" layer="96" rot="R270"/>
+</instance>
+<instance part="HV_IN" gate="G$1" x="167.64" y="-17.78" smashed="yes">
+<attribute name="NAME" x="160.00796875" y="-12.69198125" size="1.780809375" layer="95"/>
+<attribute name="VALUE" x="160.006709375" y="-22.868859375" size="1.7811" layer="96"/>
 </instance>
 </instances>
@@
 </segment>
 <segment>
-<pinref part="HV_IN" gate="G$1" pin="GNDBREAK"/>
-<wire x1="172.72" y1="-17.78" x2="182.88" y2="-17.78" width="0.1524" layer="91"/>
-<wire x1="182.88" y1="-17.78" x2="182.88" y2="-20.32" width="0.1524" layer="91"/>
+<wire x1="172.72" y1="-20.32" x2="182.88" y2="-20.32" width="0.1524" layer="91"/>
 <pinref part="GND20" gate="1" pin="GND"/>
-<pinref part="HV_IN" gate="G$1" pin="GND"/>
-<wire x1="172.72" y1="-20.32" x2="172.72" y2="-17.78" width="0.1524" layer="91"/>
-<junction x="172.72" y="-17.78"/>
+<pinref part="HV_IN" gate="G$1" pin="3"/>
+<pinref part="HV_IN" gate="G$1" pin="2"/>
+<wire x1="172.72" y1="-17.78" x2="172.72" y2="-20.32" width="0.1524" layer="91"/>
+<junction x="172.72" y="-20.32"/>
 </segment>
 <segment>
@@
 </segment>
 </net>
-<net name="N$20" class="0">
-<segment>
-<pinref part="SJ3" gate="1" pin="2"/>
-<pinref part="FEATHER" gate="G$1" pin="10"/>
-<wire x1="91.44" y1="-43.18" x2="88.9" y2="-43.18" width="0.1524" layer="91"/>
-</segment>
-</net>
 <net name="OVR_READ" class="0">
 <segment>
 <pinref part="SJ3" gate="1" pin="1"/>
-<wire x1="101.6" y1="-43.18" x2="104.14" y2="-43.18" width="0.1524" layer="91"/>
-<label x="104.14" y="-43.18" size="1.27" layer="95" xref="yes"/>
+<wire x1="116.84" y1="-43.18" x2="119.38" y2="-43.18" width="0.1524" layer="91"/>
+<label x="119.38" y="-43.18" size="1.27" layer="95" xref="yes"/>
 </segment>
 </net>
 <net name="VCC_HV" class="0">
 <segment>
-<pinref part="HV_IN" gate="G$1" pin="PWR"/>
-<wire x1="172.72" y1="-15.24" x2="182.88" y2="-15.24" width="0.1524" layer="91"/>
-<label x="182.88" y="-15.24" size="1.27" layer="95" xref="yes"/>
+<wire x1="172.72" y1="-15.24" x2="177.8" y2="-15.24" width="0.1524" layer="91"/>
+<label x="177.8" y="-15.24" size="1.27" layer="95" xref="yes"/>
+<pinref part="HV_IN" gate="G$1" pin="1"/>
 </segment>
 <segment>
@@
 </segment>
 </net>
+<net name="N$17" class="0">
+<segment>
+<pinref part="SJ3" gate="1" pin="2"/>
+<wire x1="106.68" y1="-43.18" x2="101.6" y2="-43.18" width="0.1524" layer="91"/>
+<wire x1="101.6" y1="-43.18" x2="101.6" y2="-45.72" width="0.1524" layer="91"/>
+<pinref part="FEATHER" gate="G$1" pin="9"/>
+<wire x1="101.6" y1="-45.72" x2="88.9" y2="-45.72" width="0.1524" layer="91"/>
+</segment>
+</net>
 </nets>
 </sheet>
-<sheet>
-<plain>
-</plain>
-<instances>
-</instances>
-<busses>
-</busses>
-<nets>
-</nets>
-</sheet>
